Commit message: add support for the stretch with dex wrist (more degrees of freedom)

File: urdf/stretch_description.xacro (robot description, xacro)
@@ -1,5 +1,6 @@
 <?xml version="1.0"?>
-<robot xmlns:xacro="http://www.ros.org/wiki/xacro" name="stretch">
-  <xacro:include filename="stretch_gripper.xacro" />
+<robot xmlns:xacro="http://www.ros.org/wiki/xacro" name="stretch_description">
+  <xacro:include filename="stretch_dex_wrist.xacro" />
+  <!--<xacro:include filename="stretch_gripper.xacro" /> -->
   <!--<xacro:include filename="stretch_gripper_with_puller.xacro" />-->
   <!--<xacro:include filename="stretch_dry_erase_marker.xacro" />-->

File: urdf/stretch_uncalibrated.urdf (robot description, URDF)
Before this commit: robot stretch, 42 links, 41 joints
Links:
- removed link link_grasp_center
- removed link link_gripper
- added link link_straight_gripper, mass 0.0496384234458284; collision mesh filename=package://stretch_description/meshes/link_straight_gripper.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; visual mesh filename=package://stretch_description/meshes/link_straight_gripper.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
- added link link_wrist_pitch, mass 0.0701267146295583; collision mesh filename=package://stretch_description/meshes/link_wrist_pitch.STL; visual mesh filename=package://stretch_description/meshes/link_wrist_pitch.STL
- added link link_wrist_roll, mass 0.00585666394358811; collision mesh filename=package://stretch_description/meshes/link_wrist_roll.STL; visual mesh filename=package://stretch_description/meshes/link_wrist_roll.STL
- added link link_wrist_yaw_bottom, mass 0.0988906816399982; collision mesh filename=package://stretch_description/meshes/link_wrist_yaw_bottom.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; visual mesh filename=package://stretch_description/meshes/link_wrist_yaw_bottom.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
- link link_gripper_finger_left: mass 0.0476207785199474 -> 0.0476207785199479; geometry collision mesh filename=package://stretch_description/meshes/link_gripper_finger_le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; visual mesh filename=package://stretch_description/meshes/link_gripper_finger_le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
- link link_gripper_finger_right: mass 0.0476207785199481 -> 0.047621; geometry collision mesh filename=package://stretch_description/meshes/link_gripper_finger_ri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; visual mesh filename=package://stretch_description/meshes/link_gripper_finger_ri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
- link link_gripper_fingertip_left: mass 0.00382159917455729 -> 0.00382160686584851
- link link_gripper_fingertip_right: mass 0.00382160037319545 -> 0.00382160881468841
Joints:
- removed joint joint_grasp_center
- removed joint joint_gripper
- added joint joint_straight_gripper: type fixed, parent link_wrist_roll, child link_straight_gripper, origin xyz=0 0 0.0155 rpy=3.54987407349455E-30 3.24021254484265E-20 -3.14159265358979, axis 0 0 0
- added joint joint_wrist_pitch: type revolute, parent link_wrist_yaw_bottom, child link_wrist_pitch, origin xyz=0 -0.0195500000000002 -0.0247499999999984 rpy=1.5707963267949 -8.12895570882604E-15 -3.14159265358979, axis 0 0 -1, limit lower=-1.57 upper=0.56 effort=100 velocity=1.0
- added joint joint_wrist_roll: type revolute, parent link_wrist_pitch, child link_wrist_roll, origin xyz=-0.0188587444076125 -0.0239999999998942 0.01955 rpy=3.14159265358979 1.5707963267949 0, axis 0 0 1, limit lower=-3.14 upper=3.14 effort=100 velocity=1.0
- added joint joint_wrist_yaw_bottom: type fixed, parent link_wrist_yaw, child link_wrist_yaw_bottom, origin xyz=0 0 0 rpy=-3.14159265358979 1.13367999021379E-14 1.57079632679489, axis 0 0 0
- joint joint_gripper_finger_left: axis 0 0 1 -> 0 0 -1; origin xyz=-0.047231 -0.010151 -0.04679 rpy=2.1762E-15 0.5236 3.1416 -> xyz=0.018599 0.003 0.033689 rpy=1.5708 -1.5708 0; parent link_gripper -> link_straight_gripper
- joint joint_gripper_finger_right: origin xyz=-0.047231 0.010049 -0.04679 rpy=3.1416 -0.5236 1.2943E-15 -> xyz=-0.018599 0.003 0.033689 rpy=1.5708 1.5708 0; parent link_gripper -> link_straight_gripper
- joint joint_gripper_fingertip_left: origin xyz=0.171099 0.014912 0 rpy=-1.5708 -4.774E-15 -2.5545 -> xyz=0.190596948563868 -0.015 0 rpy=1.57079632679496 4.51275387511463E-14 2.60113659715756
- joint joint_gripper_fingertip_right: origin xyz=-0.171099 -0.014912 0 rpy=-1.5708 -2.0539E-15 0.58705 -> xyz=-0.190596948563868 -0.015 0 rpy=-1.57079632679483 -3.43320051448326E-14 0.540456056432235
