Commit message: update code - get oriented bounding boxes for different geometry components

File: urdf/hab_stretch_dex_wrist_simplified.urdf (robot description, URDF)
Before this commit: robot stretch_description, 44 links, 43 joints
Links:
- link laser: geometry collision box size=0.019500 0.069940 0.069940; visual mesh filename=../meshes/laser.STL

Commit message: update numpy information for the robot

File: urdf/hab_stretch_dex_wrist_simplified.urdf (robot description, URDF)
Before this commit: robot stretch_description, 44 links, 43 joints
Links:
- link base_link: geometry collision box size=0.143197 0.324688 0.341202; visual mesh filename=../meshes/base_link.STL

Commit message: fix generation of simplified geometry + update URDF

File: urdf/hab_stretch_dex_wrist_simplified.urdf (robot description, URDF)
Before this commit: robot stretch_description, 44 links, 43 joints
Links:
- link link_mast: geometry collision box size=0.038125 0.038125 1.285000; visual mesh filename=../meshes/link_mast.STL

Commit message: create objects in a consistent way + apply a rotation to make sure appears right in habitat

File: urdf/hab_stretch_dex_wrist_simplified.urdf (robot description, URDF)
Before this commit: robot stretch_description, 44 links, 43 joints
Links:
- link base_link: mass 1.0723782659782 -> 10.0723782659782

Commit message: update urdf for the robot

File: urdf/hab_stretch_dex_wrist_simplified.urdf (robot description, URDF)
Before this commit: robot stretch_description, 44 links, 43 joints
Links:
- link base_link: geometry collision box size=0.143197 0.324688 0.361202; visual mesh filename=../meshes/base_link.STL
- link caster_link: geometry visual mesh filename=../meshes/omni_wheel_m.STL
- link link_left_wheel: geometry visual mesh filename=../meshes/link_left_wheel.STL
- link link_right_wheel: geometry visual mesh filename=../meshes/link_right_wheel.STL

Commit message: update the model - converting the dex wrist to just primitive boxes

File: urdf/hab_stretch_dex_wrist_simplified.urdf (robot description, URDF)
Before this commit: robot stretch_description, 44 links, 43 joints
Links:
- link link_straight_gripper: geometry collision box size=0.052858 0.056076 0.108538; visual mesh filename=../meshes/link_straight_gripper.STL
- link link_wrist_pitch: geometry collision box size=0.043138 0.053359 0.064888; visual mesh filename=../meshes/link_wrist_pitch.STL
- link link_wrist_roll: geometry collision box size=0.015500 0.028888 0.028987; visual mesh filename=../meshes/link_wrist_roll.STL
- link link_wrist_yaw_bottom: geometry collision box size=0.041500 0.062919 0.094300; visual mesh filename=../meshes/link_wrist_yaw_bottom.STL

Commit message: create a version made of boxes

File: urdf/hab_stretch_dex_wrist_simplified.urdf (robot description, URDF)
Before this commit: robot stretch_description, 44 links, 43 joints
Links:
- link link_arm_l0: geometry collision box size=0.059285 0.127573 0.226500; visual mesh filename=../meshes/link_arm_l0.STL
- link link_arm_l1: geometry collision box size=0.047250 0.047250 0.226500; visual mesh filename=../meshes/link_arm_l1.STL
- link link_arm_l2: geometry collision box size=0.051250 0.051250 0.226500; visual mesh filename=../meshes/link_arm_l2.STL
- link link_arm_l3: geometry collision box size=0.055250 0.055250 0.226500; visual mesh filename=../meshes/link_arm_l3.STL
- link link_arm_l4: geometry collision box size=0.059250 0.059250 0.222500; visual mesh filename=../meshes/link_arm_l4.STL
- link link_aruco_inner_wrist: geometry visual mesh filename=../meshes/link_aruco_inner_wrist.STL
- link link_aruco_left_base: geometry visual mesh filename=../meshes/link_aruco_left_base.STL
- link link_aruco_right_base: geometry visual mesh filename=../meshes/link_aruco_right_base.STL
- link link_aruco_shoulder: geometry visual mesh filename=../meshes/link_aruco_shoulder.STL
- link link_gripper_finger_left: geometry collision box size=0.013000 0.030210 0.196835; visual mesh filename=../meshes/link_gripper_finger_left.STL
- link link_gripper_finger_right: geometry collision box size=0.013000 0.030210 0.196835; visual mesh filename=../meshes/link_gripper_finger_right.STL
- link link_head: geometry collision box size=0.056453 0.131612 0.195150; visual mesh filename=../meshes/link_head.STL
- link link_head_pan: geometry collision box size=0.043969 0.048193 0.122235; visual mesh filename=../meshes/link_head_pan.STL
- link link_head_tilt: geometry collision box size=0.061014 0.068029 0.120844; visual mesh filename=../meshes/link_head_tilt.STL
- link link_lift: geometry collision box size=0.120261 0.137963 0.258855; visual mesh filename=../meshes/link_lift.STL
- link link_wrist_yaw: geometry collision box size=0.029951 0.029976 0.038000; visual mesh filename=../meshes/link_wrist_yaw.STL
- link respeaker_base: geometry collision box size=0.042669 0.070906 0.079812; visual mesh filename=../meshes/link_respeaker.STL
