Commit message: orientation change first

File: urdf/planner_stretch_dex_wrist_simplified.urdf (robot description, URDF)
Before this commit: robot stretch_description, 47 links, 46 joints
Joints:
- joint base_theta_joint: child base_link -> base_theta_link; limit (none) -> lower=-3.14159 upper=3.14159 effort=100 velocity=1.0; parent base_theta_link -> world; type continuous -> revolute
- joint base_x_joint: parent world -> base_theta_link
- joint base_y_joint: child base_theta_link -> base_link

Commit message: add new test to make sure planner makes sense

File: urdf/planner_stretch_dex_wrist_simplified.urdf (robot description, URDF)
Before this commit: robot stretch_description, 47 links, 46 joints
Joints:
- joint base_theta_joint: axis (none) -> 0 0 1

Commit message: x and y axes work in motion planning now

File: urdf/planner_stretch_dex_wrist_simplified.urdf (robot description, URDF)
Before this commit: robot stretch_description, 47 links, 46 joints
Joints:
- joint base_x_joint: origin (none) -> rpy=0 0 -1.57079632679496
- joint base_y_joint: origin (none) -> rpy=0 0 1.57079632679496

Commit message: update joint information and make sure the robot is moving around properly

File: urdf/planner_stretch_dex_wrist_simplified.urdf (robot description, URDF)
Before this commit: robot stretch_description, 47 links, 46 joints
Joints:
- joint base_x_joint: axis (none) -> 1 0 0
- joint base_y_joint: axis (none) -> 1 0 0

Commit message: update pybullet

File: urdf/planner_stretch_dex_wrist_simplified.urdf (robot description, URDF)
Before this commit: robot stretch_description, 47 links, 46 joints
Joints:
- joint base_theta_joint: origin (none) -> xyz=0 0 0 rpy=0 0 0
- joint base_x_joint: axis 1 0 0 -> (none)

Commit message: update test bullet plannet thing

File: urdf/planner_stretch_dex_wrist_simplified.urdf (robot description, URDF)
Before this commit: robot stretch_description, 47 links, 46 joints
Joints:
- joint base_x_joint: axis (none) -> 1 0 0

Commit message: make some tweaks to planner urdf - correcting references to remove angle issues

File: urdf/planner_stretch_dex_wrist_simplified.urdf (robot description, URDF)
Before this commit: robot stretch_description, 47 links, 46 joints
Joints:
- joint base_theta_joint: axis 0 0 1 -> 0 0 -1; child base_theta_link -> base_link; parent world -> base_theta_link
- joint base_x_joint: origin rpy=0 0 -1.57079632679496 -> rpy=0 0 0; parent base_theta_link -> world
- joint base_y_joint: child base_link -> base_theta_link

Commit message: fixing angle issues again

File: urdf/planner_stretch_dex_wrist_simplified.urdf (robot description, URDF)
Before this commit: robot stretch_description, 47 links, 46 joints
Joints:
- joint base_theta_joint: axis 0 0 -1 -> 0 0 1; origin xyz=0 0 0 rpy=0 0 0 -> xyz=0 0 0 rpy=0 0 -1.57079632679496
