Commit message: add imu info

File: urdf/planner_calibrated_simplified.urdf (robot description, URDF)
Before this commit: robot stretch_description, 47 links, 46 joints
Links:
- added link base_imu, mass 0.000901473198307758; collision mesh filename=package://stretch_description/meshes/base_imu.STL; visual mesh filename=package://stretch_description/meshes/base_imu.STL
Joints:
- added joint joint_base_imu: type fixed, parent base_link, child base_imu, origin xyz=-0.12838 0.0031592 0.1474 rpy=-3.1416 0 -1.5708, axis 0 0 0

Commit message: update meshes

File: urdf/planner_calibrated_simplified.urdf (robot description, URDF)
Before this commit: robot stretch_description, 48 links, 47 joints
Links:
- link base_imu: geometry collision mesh filename=../meshes/base_imu.STL; visual mesh filename=../meshes/base_imu.STL

Commit message: add imu to simplified mesh

File: urdf/planner_calibrated_simplified.urdf (robot description, URDF)
Before this commit: robot stretch_description, 47 links, 46 joints
Links:
- added link base_imu, mass 0.000901473198307758; collision mesh filename=../meshes/base_imu.STL; visual mesh filename=../meshes/base_imu.STL
Joints:
- added joint joint_base_imu: type fixed, parent base_link, child base_imu, origin xyz=-0.12838 0.0031592 0.1474 rpy=-3.1416 0 -1.5708, axis 0 0 0
