Commit message: based on crhis urdf with heavier gripper

File: urdf/hab_stretch.urdf (robot description, URDF)
Before this commit: robot stretch, 42 links, 41 joints
Links:
- removed link link_grasp_center
- removed link link_gripper
- added link link_straight_gripper, mass 0.496384234458284; collision box size=0.052858 0.056076 0.108538; visual mesh filename=../meshes/link_straight_gripper.STL
- added link link_wrist_pitch, mass 0.0701267146295583; collision box size=0.043138 0.053359 0.064888; visual mesh filename=../meshes/link_wrist_pitch.STL
- added link link_wrist_roll, mass 0.00585666394358811; collision box size=0.015500 0.028888 0.028987; visual mesh filename=../meshes/link_wrist_roll.STL
- added link link_wrist_yaw_bottom, mass 0.0988906816399982; collision box size=0.041500 0.062919 0.094300; visual mesh filename=../meshes/link_wrist_yaw_bottom.STL
- link base_link: mass 1.0723782659782 -> 10.0723782659782; geometry collision box size=0.123197 0.304688 0.361202; visual mesh filename=../meshes/base_link.obj
- link caster_link: geometry collision sphere radius=0.032; visual mesh filename=../meshes/omni_wheel_m.obj
- link laser: geometry collision box size=0.019500 0.069940 0.069940; visual mesh filename=../meshes/laser.obj
- link link_arm_l0: mass 0.101241250325294 -> 1.01241250325294; geometry collision box size=0.059285 0.127573 0.226500; visual mesh filename=../meshes/link_arm_l0.obj
- link link_arm_l1: mass 0.0511763619538321 -> 0.511763619538321; geometry collision box size=0.047250 0.047250 0.226500; visual mesh filename=../meshes/link_arm_l1.obj
- link link_arm_l2: mass 0.0569074368576238 -> 0.569074368576238; geometry collision box size=0.051250 0.051250 0.226500; visual mesh filename=../meshes/link_arm_l2.obj
- link link_arm_l3: mass 0.0626921047058405 -> 0.626921047058405; geometry collision box size=0.055250 0.055250 0.226500; visual mesh filename=../meshes/link_arm_l3.obj
- link link_arm_l4: mass 0.0676525455789735 -> 0.676525455789735; geometry collision box size=0.059250 0.059250 0.222500; visual mesh filename=../meshes/link_arm_l4.obj
- link link_aruco_inner_wrist: geometry visual mesh filename=../meshes/link_aruco_inner_wrist.STL
- link link_aruco_left_base: geometry visual mesh filename=../meshes/link_aruco_left_base.STL
- link link_aruco_right_base: geometry visual mesh filename=../meshes/link_aruco_right_base.STL
- link link_aruco_shoulder: geometry visual mesh filename=../meshes/link_aruco_shoulder.STL
- link link_gripper_finger_left: mass 0.0476207785199474 -> 4.76207785199479; geometry collision box size=0.013000 0.030210 0.196835; visual mesh filename=../meshes/link_gripper_finger_left.obj
- link link_gripper_finger_right: mass 0.0476207785199481 -> 4.7621; geometry collision box size=0.013000 0.030210 0.196835; visual mesh filename=../meshes/link_gripper_finger_right.obj
- link link_gripper_fingertip_left: mass 0.00382159917455729 -> 0.00382160686584851; geometry collision mesh filename=../meshes/link_gripper_fingertip_left.obj; visual mesh filename=../meshes/link_gripper_fingertip_left.obj
- link link_gripper_fingertip_right: mass 0.00382160037319545 -> 0.00382160881468841; geometry collision mesh filename=../meshes/link_gripper_fingertip_right.obj; visual mesh filename=../meshes/link_gripper_fingertip_right.obj
- link link_head: geometry collision box size=0.056453 0.131612 0.195150; visual mesh filename=../meshes/link_head.obj
- link link_head_pan: geometry collision box size=0.043969 0.048193 0.122235; visual mesh filename=../meshes/link_head_pan.obj
- link link_head_tilt: geometry collision box size=0.061014 0.068029 0.120844; visual mesh filename=../meshes/link_head_tilt.obj
- link link_left_wheel: geometry collision cylinder length=0.04 radius=0.05; visual mesh filename=../meshes/link_left_wheel.obj
- link link_lift: geometry collision box size=0.120261 0.127963 0.238855; visual mesh filename=../meshes/link_lift.obj
- link link_mast: geometry collision box size=0.038125 0.038125 1.285000; visual mesh filename=../meshes/link_mast.obj
- link link_right_wheel: geometry collision cylinder length=0.04 radius=0.05; visual mesh filename=../meshes/link_right_wheel.obj
- link link_wrist_yaw: geometry collision box size=0.029951 0.029976 0.038000; visual mesh filename=../meshes/link_wrist_yaw.obj
- link respeaker_base: geometry collision box size=0.042669 0.070906 0.079812; visual mesh filename=../meshes/link_respeaker.obj
Joints:
- removed joint joint_grasp_center
- removed joint joint_gripper
- added joint joint_straight_gripper: type fixed, parent link_wrist_roll, child link_straight_gripper, origin xyz=0 0 0.0155 rpy=3.54987407349455E-30 3.24021254484265E-20 -3.14159265358979, axis 0 0 0
- added joint joint_wrist_pitch: type revolute, parent link_wrist_yaw_bottom, child link_wrist_pitch, origin xyz=0 -0.0195500000000002 -0.0247499999999984 rpy=1.5707963267949 -8.12895570882604E-15 -3.14159265358979, axis 0 0 -1, limit lower=-1.57 upper=0.56 effort=100 velocity=1.0
- added joint joint_wrist_roll: type revolute, parent link_wrist_pitch, child link_wrist_roll, origin xyz=-0.0188587444076125 -0.0239999999998942 0.01955 rpy=3.14159265358979 1.5707963267949 0, axis 0 0 1, limit lower=-3.14 upper=3.14 effort=100 velocity=1.0
- added joint joint_wrist_yaw_bottom: type fixed, parent link_wrist_yaw, child link_wrist_yaw_bottom, origin xyz=0 0 0 rpy=-3.14159265358979 1.13367999021379E-14 1.57079632679489, axis 0 0 0
- joint joint_gripper_finger_left: axis 0 0 1 -> 0 0 -1; origin xyz=-0.047231 -0.010151 -0.04679 rpy=2.1762E-15 0.5236 3.1416 -> xyz=0.018599 0.003 0.033689 rpy=1.5708 -1.5708 0; parent link_gripper -> link_straight_gripper
- joint joint_gripper_finger_right: origin xyz=-0.047231 0.010049 -0.04679 rpy=3.1416 -0.5236 1.2943E-15 -> xyz=-0.018599 0.003 0.033689 rpy=1.5708 1.5708 0; parent link_gripper -> link_straight_gripper
- joint joint_gripper_fingertip_left: origin xyz=0.171099 0.014912 0 rpy=-1.5708 -4.774E-15 -2.5545 -> xyz=0.190596948563868 -0.015 0 rpy=1.57079632679496 4.51275387511463E-14 2.60113659715756
- joint joint_gripper_fingertip_right: origin xyz=-0.171099 -0.014912 0 rpy=-1.5708 -2.0539E-15 0.58705 -> xyz=-0.190596948563868 -0.015 0 rpy=-1.57079632679483 -3.43320051448326E-14 0.540456056432235

Commit message: make gripper heavy

File: urdf/hab_stretch.urdf (robot description, URDF)
Before this commit: robot stretch, 42 links, 41 joints
Links:
- link base_link: mass 1.0723782659782 -> 10.0723782659782
- link link_arm_l0: mass 0.101241250325294 -> 1.01241250325294
- link link_arm_l1: mass 0.0511763619538321 -> 0.511763619538321
- link link_arm_l2: mass 0.0569074368576238 -> 0.569074368576238
- link link_arm_l3: mass 0.0626921047058405 -> 0.626921047058405
- link link_arm_l4: mass 0.0676525455789735 -> 0.676525455789735
- link link_gripper_finger_left: mass 0.0476207785199474 -> 4.76207785199474
- link link_gripper_finger_right: mass 0.0476207785199481 -> 4.76207785199481

Commit message: make heavy for gripper

File: urdf/hab_stretch.urdf (robot description, URDF)
Before this commit: robot stretch, 42 links, 41 joints
Links:
- link link_arm_l4: mass 0.676525455789735 -> 0.676525455789736
