Commit message: update urdf for my robot

File: urdf/planner_calibrated_manipulation_mode.urdf (robot description, URDF)
Before this commit: robot stretch_description, 47 links, 46 joints
Links:
- link base_link: mass 10.0723782659782 -> 1.1912; geometry collision mesh filename=package://stretch_description/meshes/base_link.STL; visual mesh filename=package://stretch_description/meshes/base_link.STL
- link camera_link: geometry collision box size=0.02505 0.09 0.025; visual mesh filename=package://realsense2_description/meshes/d435.dae
- link caster_link: geometry collision sphere radius=0.032; visual mesh filename=package://stretch_description/meshes/omni_wheel_m.STL
- link laser: geometry collision mesh filename=package://stretch_description/meshes/laser.STL; visual mesh filename=package://stretch_description/meshes/laser.STL
- link link_arm_l0: mass 0.101241250325294 -> 0.085003260946398; geometry collision mesh filename=package://stretch_description/meshes/link_arm_l0.STL; visual mesh filename=package://stretch_description/meshes/link_arm_l0.STL
- link link_arm_l1: mass 0.0511763619538321 -> 0.051382; geometry collision mesh filename=package://stretch_description/meshes/link_arm_l1.STL; visual mesh filename=package://stretch_description/meshes/link_arm_l1.STL
- link link_arm_l2: mass 0.0569074368576238 -> 0.0571386353275368; geometry collision mesh filename=package://stretch_description/meshes/link_arm_l2.STL; visual mesh filename=package://stretch_description/meshes/link_arm_l2.STL
- link link_arm_l3: mass 0.0626921047058405 -> 0.0628927381893134; geometry collision mesh filename=package://stretch_description/meshes/link_arm_l3.STL; visual mesh filename=package://stretch_description/meshes/link_arm_l3.STL
- link link_arm_l4: mass 0.0676525455789735 -> 0.068095; geometry collision mesh filename=package://stretch_description/meshes/link_arm_l4.STL; visual mesh filename=package://stretch_description/meshes/link_arm_l4.STL
- link link_aruco_inner_wrist: geometry collision mesh filename=package://stretch_description/meshes/link_aruco_inner_wrist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; visual mesh filename=package://stretch_description/meshes/link_aruco_inner_wrist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
- link link_aruco_left_base: geometry collision mesh filename=package://stretch_description/meshes/link_aruco_left_base.S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; visual mesh filename=package://stretch_description/meshes/link_aruco_left_base.S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
- link link_aruco_right_base: geometry collision mesh filename=package://stretch_description/meshes/link_aruco_right_base.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; visual mesh filename=package://stretch_description/meshes/link_aruco_right_base.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
- link link_aruco_shoulder: geometry collision mesh filename=package://stretch_description/meshes/link_aruco_shoulder.STL; visual mesh filename=package://stretch_description/meshes/link_aruco_shoulder.STL
- link link_aruco_top_wrist: geometry collision mesh filename=package://stretch_description/meshes/link_aruco_top_wrist.S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; visual mesh filename=package://stretch_description/meshes/link_aruco_top_wrist.S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
- link link_gripper_finger_left: geometry collision mesh filename=package://stretch_description/meshes/link_gripper_finger_le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; visual mesh filename=package://stretch_description/meshes/link_gripper_finger_le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
- link link_gripper_finger_right: geometry collision mesh filename=package://stretch_description/meshes/link_gripper_finger_ri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; visual mesh filename=package://stretch_description/meshes/link_gripper_finger_ri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
- link link_gripper_fingertip_left: geometry collision mesh filename=package://stretch_description/meshes/link_gripper_fingertip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; visual mesh filename=package://stretch_description/meshes/link_gripper_fingertip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
- link link_gripper_fingertip_right: geometry collision mesh filename=package://stretch_description/meshes/link_gripper_fingertip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; visual mesh filename=package://stretch_description/meshes/link_gripper_fingertip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
- link link_head: mass 0.129454717596498 -> 0.133027236718691; geometry collision mesh filename=package://stretch_description/meshes/link_head.STL; visual mesh filename=package://stretch_description/meshes/link_head.STL
- link link_head_pan: mass 0.035858341182617 -> 0.0273764496535409; geometry collision mesh filename=package://stretch_description/meshes/link_head_pan.STL; visual mesh filename=package://stretch_description/meshes/link_head_pan.STL
- link link_head_tilt: mass 0.0701242408063442 -> 0.090217113313934; geometry collision mesh filename=package://stretch_description/meshes/link_head_tilt.STL; visual mesh filename=package://stretch_description/meshes/link_head_tilt.STL
- link link_left_wheel: mass 0.01 -> 0.0042721; geometry collision mesh filename=package://stretch_description/meshes/link_left_wheel.STL; visual mesh filename=package://stretch_description/meshes/link_left_wheel.STL
- link link_lift: mass 0.444820831236007 -> 0.27218; geometry collision mesh filename=package://stretch_description/meshes/link_lift.STL; visual mesh filename=package://stretch_description/meshes/link_lift.STL
- link link_mast: mass 0.749143203376401 -> 1.8285; geometry collision mesh filename=package://stretch_description/meshes/link_mast.STL; visual mesh filename=package://stretch_description/meshes/link_mast.STL
- link link_right_wheel: mass 0.01 -> 0.0042721; geometry collision mesh filename=package://stretch_description/meshes/link_right_wheel.STL; visual mesh filename=package://stretch_description/meshes/link_right_wheel.STL
- link link_straight_gripper: geometry collision mesh filename=package://stretch_description/meshes/link_straight_gripper.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; visual mesh filename=package://stretch_description/meshes/link_straight_gripper.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
- link link_wrist_pitch: geometry collision mesh filename=package://stretch_description/meshes/link_wrist_pitch.STL; visual mesh filename=package://stretch_description/meshes/link_wrist_pitch.STL
- link link_wrist_roll: geometry collision mesh filename=package://stretch_description/meshes/link_wrist_roll.STL; visual mesh filename=package://stretch_description/meshes/link_wrist_roll.STL
- link link_wrist_yaw: mass 0.0405398981326229 -> 0.0404746907425003; geometry collision mesh filename=package://stretch_description/meshes/link_wrist_yaw.STL; visual mesh filename=package://stretch_description/meshes/link_wrist_yaw.STL
- link link_wrist_yaw_bottom: geometry collision mesh filename=package://stretch_description/meshes/link_wrist_yaw_bottom.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; visual mesh filename=package://stretch_description/meshes/link_wrist_yaw_bottom.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
- link respeaker_base: mass 0.00969129410417277 -> 0.015643; geometry collision mesh filename=package://stretch_description/meshes/respeaker_base.STL; visual mesh filename=package://stretch_description/meshes/respeaker_base.STL
Joints:
- joint base_theta_joint: limit lower=0.0 upper=0.0 effort=100.0 velocity=1.0 -> (none); origin xyz=0.0 0.0 0.0 rpy=0.0 0.0 -1.57079632679496 -> xyz=0.0 0.0 0.0 rpy=0.0 0.0 0.0
- joint base_y_joint: limit lower=0.0 upper=0.0 effort=100.0 velocity=3.0 -> (none); origin xyz=0 0 0 rpy=0.0 0.0 1.57079632679496 -> xyz=0 0 0 rpy=0.0 0.0 0.0
- joint camera_joint: origin xyz=0.025070381118864622 -0.012287278361953074 0.017905872362600883 rpy=0.0027184810411859444 0.001558563349419062 -0.04777120277132254 -> xyz=0.02802960503838624 -0.007608222297947431 0.018218494141479257 rpy=0.010658876360659654 -0.0022761048951753793 0.018675317090921212
- joint joint_arm_l0: origin xyz=0.0 0.0 -0.0137499999999938 rpy=-3.05317390622457e-16 -4.23236224076729e-16 -2.68425135229209e-17 -> xyz=0.0 0.0 -0.0137499999991968 rpy=7.63746778746202e-30 -3.80121128864402e-15 2.62707547767438e-15
- joint joint_arm_l1: origin xyz=0.0 0.0 0.013 rpy=7.41596560408007e-17 1.33876788296791e-16 -2.44545873596083e-16 -> xyz=0.0 0.0 0.0129999999999981 rpy=-7.63746778746202e-30 -7.88860905221012e-31 1.11022302462516e-16
- joint joint_arm_l2: origin xyz=0.0 0.0 0.013 rpy=2.91385731014123e-16 4.44300759504684e-17 3.25691080516352e-16 -> xyz=0.0 0.0 0.013 rpy=0.0 1.57655765344625e-30 -1.66533453693773e-16
- joint joint_arm_l3: origin xyz=0.0 0.0 0.013 rpy=3.5742e-16 3.2123e-16 -2.4565e-16 -> xyz=0.0 0.0 0.013 rpy=7.68831233799385e-30 2.36716479416092e-30 2.29652732251143e-17
- joint joint_arm_l4: origin xyz=-0.25669443874094205 0.005713417002918588 0.0012296937814473496 rpy=1.5781652616599324 0.04551858006017695 -1.6181874684011688 -> xyz=-0.25956015433181046 -0.0059261537843136765 -0.005557384627505743 rpy=1.5619286973774569 -0.006924580188019336 -1.575847166561953
- joint joint_aruco_right_base: origin xyz=-0.00500000000000014 -0.1304972 0.1597482 rpy=0.0 0.0 -1.5707963267949 -> xyz=-0.0015028 -0.1304972 0.1597482 rpy=0.0 0.0 -1.5707963267949
- joint joint_head: origin xyz=0.0 1.33 0.0 rpy=1.5708 -1.5615 3.1416 -> xyz=0.0 1.33 0.0 rpy=1.5707963267949 -1.5707963267949 3.1416
- joint joint_head_pan: origin xyz=0.14394738959044898 0.0689269242761915 -0.003064182445303723 rpy=0.008083283195200545 0.000583944763831834 1.620778470351339 -> xyz=0.1284513021260868 0.07637128403435504 0.00023722543808071166 rpy=-0.013467967166369273 0.005690738105448956 1.6024957766579377
- joint joint_head_tilt: origin xyz=-0.0038009318349181698 0.027661869381952295 -0.06046636278717248 rpy=1.583686486584009 0.038258710433179965 0.07682454066916562 -> xyz=0.0032337815907659225 0.030910701770693223 -0.04783143162927699 rpy=1.5763332066189244 -0.029319157204454882 -0.005080558641851002
- joint joint_laser: origin xyz=0.000502800000000914 0.0 0.1664 rpy=0.0 0.0 -3.14159265358979 -> xyz=0.004 0.0 0.1664 rpy=0.0 0.0 3.1416
- joint joint_left_wheel: origin xyz=-0.00300000000001899 0.15765 0.0507999999999994 rpy=-1.5707963267949 3.16227047920818e-31 7.88745438253713e-16 -> xyz=0.0 0.17035 0.0508 rpy=-1.5708 2.6317e-16 -8.2057e-19
- joint joint_lift: origin xyz=-0.0369217062323472 0.165471199999996 -0.000341653286793524 rpy=-1.57079632679552 1.5615431375292 -6.2942004366467e-13 -> xyz=-0.037385 0.1666 0.0 rpy=-1.5708 1.5708 0.0
- joint joint_mast: origin xyz=-0.06949477028757628 0.13838980304778414 0.027045430913364362 rpy=1.5646590837134537 -0.017304958691331196 0.04825274364916361 -> xyz=-0.07174416574437388 0.13780491000396983 0.03663931715774088 rpy=1.5780076046568878 0.016499709009588637 -0.007971437955302632
- joint joint_respeaker: origin xyz=1.09074743137871e-05 1.36992 0.00303572796911382 rpy=1.57079632679553 0.0 3.14159265358916 -> xyz=0.0 1.37236408874452 0.00303065898329655 rpy=-1.5707963267949 -0.698131700797725 4.93295812652799e-16
- joint joint_right_wheel: origin xyz=-0.00300000000000034 -0.15765 0.0508000000000004 rpy=-1.57079632679489 -1.11022302462516e-16 7.28583859910277e-17 -> xyz=0.0 -0.17035 0.0508 rpy=-1.5708 1.2717e-16 4.8006e-17
- joint joint_wrist_yaw: origin xyz=0.083 -0.03075 0.0 rpy=1.5708 4.2595e-14 2.6415e-15 -> xyz=0.0830000000000654 -0.0307500000000129 0.0 rpy=1.5708 4.2595e-14 2.6415e-15

Commit message: fix urdf paths

File: urdf/planner_calibrated_manipulation_mode.urdf (robot description, URDF)
Before this commit: robot stretch_description, 47 links, 46 joints
Links:
- link base_link: geometry collision mesh filename=../meshes/base_link.STL; visual mesh filename=../meshes/base_link.STL
- link caster_link: geometry collision sphere radius=0.032; visual mesh filename=../meshes/omni_wheel_m.STL
- link laser: geometry collision mesh filename=../meshes/laser.STL; visual mesh filename=../meshes/laser.STL
- link link_arm_l0: geometry collision mesh filename=../meshes/link_arm_l0.STL; visual mesh filename=../meshes/link_arm_l0.STL
- link link_arm_l1: geometry collision mesh filename=../meshes/link_arm_l1.STL; visual mesh filename=../meshes/link_arm_l1.STL
- link link_arm_l2: geometry collision mesh filename=../meshes/link_arm_l2.STL; visual mesh filename=../meshes/link_arm_l2.STL
- link link_arm_l3: geometry collision mesh filename=../meshes/link_arm_l3.STL; visual mesh filename=../meshes/link_arm_l3.STL
- link link_arm_l4: geometry collision mesh filename=../meshes/link_arm_l4.STL; visual mesh filename=../meshes/link_arm_l4.STL
- link link_aruco_inner_wrist: geometry collision mesh filename=../meshes/link_aruco_inner_wrist.STL; visual mesh filename=../meshes/link_aruco_inner_wrist.STL
- link link_aruco_left_base: geometry collision mesh filename=../meshes/link_aruco_left_base.STL; visual mesh filename=../meshes/link_aruco_left_base.STL
- link link_aruco_right_base: geometry collision mesh filename=../meshes/link_aruco_right_base.STL; visual mesh filename=../meshes/link_aruco_right_base.STL
- link link_aruco_shoulder: geometry collision mesh filename=../meshes/link_aruco_shoulder.STL; visual mesh filename=../meshes/link_aruco_shoulder.STL
- link link_aruco_top_wrist: geometry collision mesh filename=../meshes/link_aruco_top_wrist.STL; visual mesh filename=../meshes/link_aruco_top_wrist.STL
- link link_gripper_finger_left: geometry collision mesh filename=../meshes/link_gripper_finger_left.STL; visual mesh filename=../meshes/link_gripper_finger_left.STL
- link link_gripper_finger_right: geometry collision mesh filename=../meshes/link_gripper_finger_right.STL; visual mesh filename=../meshes/link_gripper_finger_right.STL
- link link_gripper_fingertip_left: geometry collision mesh filename=../meshes/link_gripper_fingertip_left.STL; visual mesh filename=../meshes/link_gripper_fingertip_left.STL
- link link_gripper_fingertip_right: geometry collision mesh filename=../meshes/link_gripper_fingertip_right.STL; visual mesh filename=../meshes/link_gripper_fingertip_right.STL
- link link_head: geometry collision mesh filename=../meshes/link_head.STL; visual mesh filename=../meshes/link_head.STL
- link link_head_pan: geometry collision mesh filename=../meshes/link_head_pan.STL; visual mesh filename=../meshes/link_head_pan.STL
- link link_head_tilt: geometry collision mesh filename=../meshes/link_head_tilt.STL; visual mesh filename=../meshes/link_head_tilt.STL
- link link_left_wheel: geometry collision mesh filename=../meshes/link_left_wheel.STL; visual mesh filename=../meshes/link_left_wheel.STL
- link link_lift: geometry collision mesh filename=../meshes/link_lift.STL; visual mesh filename=../meshes/link_lift.STL
- link link_mast: geometry collision mesh filename=../meshes/link_mast.STL; visual mesh filename=../meshes/link_mast.STL
- link link_right_wheel: geometry collision mesh filename=../meshes/link_right_wheel.STL; visual mesh filename=../meshes/link_right_wheel.STL
- link link_straight_gripper: geometry collision mesh filename=../meshes/link_straight_gripper.STL; visual mesh filename=../meshes/link_straight_gripper.STL
- link link_wrist_pitch: geometry collision mesh filename=../meshes/link_wrist_pitch.STL; visual mesh filename=../meshes/link_wrist_pitch.STL
- link link_wrist_roll: geometry collision mesh filename=../meshes/link_wrist_roll.STL; visual mesh filename=../meshes/link_wrist_roll.STL
- link link_wrist_yaw: geometry collision mesh filename=../meshes/link_wrist_yaw.STL; visual mesh filename=../meshes/link_wrist_yaw.STL
- link link_wrist_yaw_bottom: geometry collision mesh filename=../meshes/link_wrist_yaw_bottom.STL; visual mesh filename=../meshes/link_wrist_yaw_bottom.STL
- link respeaker_base: geometry collision mesh filename=../meshes/respeaker_base.STL; visual mesh filename=../meshes/respeaker_base.STL

Commit message: update URDF for the new robot

File: urdf/planner_calibrated_manipulation_mode.urdf (robot description, URDF)
Before this commit: robot stretch_description, 47 links, 46 joints
Links:
- link camera_link: geometry collision box size=0.02505 0.09 0.025; visual mesh filename=meshes/realsense2/d435.dae
