Commit message: debug habitat urdf + improve physics

File: habitat_stretch/urdf/hab_stretch.urdf (robot description, URDF)
Before this commit: robot stretch_description, 44 links, 43 joints
Links:
- link base_link: geometry collision box size=0.123197 0.284688 0.361202; visual mesh filename=../meshes/base_link.obj
- link caster_link: geometry collision sphere radius=0.032; visual mesh filename=../meshes/omni_wheel_m.obj
- link link_left_wheel: geometry collision mesh filename=../meshes/link_left_wheel.STL; visual mesh filename=../meshes/link_left_wheel.obj
- link link_right_wheel: geometry collision mesh filename=../meshes/link_right_wheel.STL; visual mesh filename=../meshes/link_right_wheel.obj

Commit message: switch to using primitives for the wheels

File: habitat_stretch/urdf/hab_stretch.urdf (robot description, URDF)
Before this commit: robot stretch_description, 44 links, 43 joints
Links:
- link link_left_wheel: geometry collision cylinder length=0.04 radius=0.05; visual mesh filename=../meshes/link_left_wheel.obj
- link link_right_wheel: geometry collision cylinder length=0.04 radius=0.05; visual mesh filename=../meshes/link_right_wheel.obj

Commit message: more collision geometry tweaks - make the robot a bit better

File: habitat_stretch/urdf/hab_stretch.urdf (robot description, URDF)
Before this commit: robot stretch_description, 44 links, 43 joints
Links:
- link base_link: geometry collision box size=0.123197 0.304688 0.361202; visual mesh filename=../meshes/base_link.obj
- link link_lift: geometry collision box size=0.120261 0.127963 0.238855; visual mesh filename=../meshes/link_lift.obj

Commit message: update habitat stretch setup

File: habitat_stretch/urdf/hab_stretch.urdf (robot description, URDF)
Before this commit: robot stretch_description, 44 links, 43 joints
Links:
- link caster_link: geometry visual mesh filename=../meshes/omni_wheel_m.obj
- link link_left_wheel: geometry visual mesh filename=../meshes/link_left_wheel.obj
- link link_right_wheel: geometry visual mesh filename=../meshes/link_right_wheel.obj
